File: motor-imu-cape.brd (EAGLE design)
At the start: 54.3 x 58.4 mm, 20 parts, among them IC1 40109, IC2 40109, IC3 24LC256P

Commit message: Final layout changes for submission to oshpark for fab.
Parts:
- renumbered JP1 to ADDR, JP2 to V_ENCODER, SV10 to PWM2, SV11 to QEP0, SV12 to QEP1, SV13 to QEP2, SV7 to GY-521, SV8 to PWM0, SV9 to PWM1
Other:
- board text removed: "GY-521"
- board text removed: "PWM0"
- board text removed: "QEP0"
- board text removed: "V ENCODER"
