File: motor-imu-cape.sch (EAGLE design)
At the start: 20 parts, among them IC1 40109, IC2 40109, IC3 24LC256P

Commit message: Final layout changes for submission to oshpark for fab.
Parts:
- renumbered JP1 to ADDR, JP2 to V_ENCODER, SV10 to PWM2, SV11 to QEP0, SV12 to QEP1, SV13 to QEP2, SV7 to GY-521, SV8 to PWM0, SV9 to PWM1
